File: PCB/MotorcycleSpeedometer.kicad_pcb (KiCad board)
At the start: 2 copper layers, 7 parts, among them J1 Conn_ARM_JTAG_SWD_10, Q1 2N7002, Q2 2N7002, Q3 2N7002, Q4 2N7002, Q5 2N7002, U1 MDBT42Q-512K

Commit message: Updated PCB
Parts:
- removed U1: MDBT42Q-512K, RF_Module:Raytac_MDBT42Q
- added C1: 10uF, Capacitor_SMD:C_0603_1608Metric, F.Cu at (82.5, 76.9)
- added C2: 100nF, Capacitor_SMD:C_0603_1608Metric, F.Cu at (82.5, 79.4)
- added C3: 100nF, Capacitor_SMD:C_0603_1608Metric, F.Cu at (82.5, 81.9)
- added C4: 100nF, Capacitor_SMD:C_0603_1608Metric, F.Cu at (82.5, 84.4)
- added C5: 100nF, Capacitor_SMD:C_0603_1608Metric, F.Cu at (82.5, 86.9)
- added IC1: STM32U083CCT6, MyFootprints:QFP50P900X900X160-48N, F.Cu at (82.6, 57.9)
- added R1: R, Resistor_SMD:R_0603_1608Metric, F.Cu at (82.5, 89.4)
- added R10: R, Resistor_SMD:R_0603_1608Metric, F.Cu at (90.6, 81.9)
- added R2: R, Resistor_SMD:R_0603_1608Metric, F.Cu at (86.6, 76.9)
- added R3: R, Resistor_SMD:R_0603_1608Metric, F.Cu at (86.6, 79.4)
- added R4: R, Resistor_SMD:R_0603_1608Metric, F.Cu at (86.6, 81.9)
- added R5: R, Resistor_SMD:R_0603_1608Metric, F.Cu at (86.6, 84.4)
- added R6: R, Resistor_SMD:R_0603_1608Metric, F.Cu at (86.6, 86.9)
- added R7: R, Resistor_SMD:R_0603_1608Metric, F.Cu at (86.6, 89.4)
- added R8: R, Resistor_SMD:R_0603_1608Metric, F.Cu at (90.6, 76.9)
- added R9: R, Resistor_SMD:R_0603_1608Metric, F.Cu at (90.6, 79.4)
- J1: value Conn_ARM_JTAG_SWD_10 -> Conn_02x08_Odd_Even; footprint Connector_PinHeader_1.27mm:PinHeader_2x05_P1.27mm_Vertical -> Connector_PinHeader_2.54mm:PinHeader_2x08_P2.54mm_Vertical
- Q4, Q5: value 2N7002 -> AO3401A
- moved J1 49.1 mm to (75.7, 77.9), turned to 0 degrees
- moved Q4 15.6 mm to (61.9, 53.8)
- moved Q5 14.0 mm to (62.2, 60.6)
- moved Q3 6.06 mm to (51.9, 67.6)
- moved Q2 2.54 mm to (52.4, 59.4)
Connections:
- J1 pad 1: +3.3V -> +BATT
- J1 pad 10: Net-(J1-~{RESET}) -> /IGNITION_EXT
- J1 pad 2: Net-(J1-SWDIO/TMS) -> +6V
- J1 pad 3: GND -> /RTURN_EXT
- J1 pad 4: Net-(J1-SWCLK/TCK) -> unconnected-(J1-Pin_4-Pad4)
- J1 pad 5: GND -> /LTURN_EXT
- J1 pad 6: unconnected-(J1-SWO/TDO-Pad6) -> GND
- J1 pad 7: unconnected-(J1-KEY-Pad7) -> /BEAM_EXT
- J1 pad 9: GND -> /LED_EXT
- Q4 pad 3: +3.3V -> +BATT
- Q5 pad 3: +3.3V -> +BATT
